Commit message: Added in Gazebo.

File: urdf/orbit_bot.urdf (robot description, URDF)
Before this commit: robot orbit_bot, 5 links, 4 joints
Links:
- link base_link: mass None -> 0.001; geometry collision box size=0.5 0.3 0.1; visual box size=0.5 0.3 0.1
- link caster_wheel: mass None -> 0.2; geometry collision sphere radius=0.05; visual sphere radius=0.05
- link left_wheel: mass None -> 0.5; geometry collision cylinder length=0.05 radius=0.1; visual cylinder length=0.05 radius=0.1
- link lidar_link: mass None -> 0.2; geometry collision cylinder length=0.08 radius=0.06; visual cylinder length=0.08 radius=0.06
- link right_wheel: mass None -> 0.5; geometry collision cylinder length=0.05 radius=0.1; visual cylinder length=0.05 radius=0.1
