Commit message: branch for vision

File: urdf/orbit_bot.urdf (robot description, URDF)
Before this commit: robot orbit_bot, 6 links, 5 joints
Links:
- added link camera_link, mass 0.1; collision box size=0.05 0.1 0.05; visual box size=0.05 0.1 0.05
- added link camera_link_optical
Joints:
- added joint camera_joint: type fixed, parent base_link, child camera_link, origin xyz=0.25 0 0.05 rpy=0 0 0
- added joint camera_optical_joint: type fixed, parent camera_link, child camera_link_optical, origin xyz=0 0 0 rpy=-1.5708 0 -1.5708
